File: hardware/esp_home_sensor/charger.kicad_sch (KiCad schematic)
At the start: 13 parts, among them U1 BQ25170

Commit message: minor update
Parts:
- added JP8: SolderJumper_2_Bridged, Jumper:SolderJumper-2_P1.3mm_Bridged2Bar_Pad1.0x1.5mm, symbol Jumper:SolderJumper_2_Bridged
- JP6: footprint (none) -> Jumper:SolderJumper-2_P1.3mm_Bridged2Bar_Pad1.0x1.5mm
Connections:
- net VOUT: now also JP8.2 (B); no longer R3.2, R4.2, U1.8 (OUT)
- new net: JP8.1 (A), R3.2, R4.2, U1.8 (OUT)
Changed lines of the file:
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@@
+	)
+	(junction
+		(at 72.39 151.13)
+		(diameter 0)
+		(color 0 0 0 0)
+	)
+	(junction
+		(at 85.09 151.13)
+		(diameter 0)
+		(color 0 0 0 0)
 	)
 	(junction
@@
 		(color 0 0 0 0)
 	)
-	(junction
-		(at 72.39 151.13)
-		(diameter 0)
-		(color 0 0 0 0)
-	)
-	(junction
-		(at 85.09 151.13)
-		(diameter 0)
-		(color 0 0 0 0)
-	)
 	(wire
 		(pts
@@
 	(wire
 		(pts
+			(xy 125.73 73.66) (xy 132.08 73.66)
+		)
+		(stroke
+			(width 0)
+			(type default)
+		)
+	)
+	(wire
+		(pts
 			(xy 72.39 151.13) (xy 72.39 153.67)
 		)
@@
 	(wire
 		(pts
+			(xy 142.24 73.66) (xy 147.32 73.66)
+		)
+		(stroke
+			(width 0)
+			(type default)
+		)
+	)
+	(wire
+		(pts
 			(xy 68.58 80.01) (xy 68.58 76.2)
 		)
@@
 		(pts
 			(xy 59.69 87.63) (xy 59.69 90.17)
-		)
-		(stroke
-			(width 0)
-			(type default)
-		)
-	)
-	(wire
-		(pts
-			(xy 125.73 73.66) (xy 147.32 73.66)
 		)
 		(stroke
@@
 	)
 	(image
-		(at 151.13 55.88)
+		(at 151.13 48.26)
 		(data "iVBORw0KGgoAAAANSUhEUgAABC4AAAFmCAYAAACiHNsAAAAABHNCSVQICAgIfAhkiAAAIABJREFU"
 			"eJzs3U+MI+ed3/8PvV7MeJOsxkmAmYUXKFqYQReBANNGDpoEAiRDhypJh2mdhrxY7USB2gsErFkd"
@@
 	)
 	(symbol
+		(lib_id "Jumper:SolderJumper_2_Bridged")
+		(at 137.16 73.66 0)
+		(unit 1)
+		(body_style 1)
+		(exclude_from_sim no)
+		(in_bom no)
+		(on_board yes)
+		(in_pos_files yes)
+		(dnp no)
+		(fields_autoplaced yes)
+		(property "Reference" "JP8"
+			(at 137.16 67.31 0)
+			(show_name no)
+			(do_not_autoplace no)
+			(effects
+				(font
+					(size 1.27 1.27)
+				)
+			)
+		)
+		(property "Value" "SolderJumper_2_Bridged"
+			(at 137.16 69.85 0)
+			(show_name no)
+			(do_not_autoplace no)
+			(effects
+				(font
+					(size 1.27 1.27)
+				)
+			)
+		)
+		(property "Footprint" "Jumper:SolderJumper-2_P1.3mm_Bridged2Bar_Pad1.0x1.5mm"
+			(at 137.16 73.66 0)
+			(hide yes)
+			(show_name no)
+			(do_not_autoplace no)
+			(effects
+				(font
+					(size 1.27 1.27)
+				)
+			)
+		)
+		(property "Datasheet" ""
+			(at 137.16 80.01 0)
+			(hide yes)
+			(show_name no)
+			(do_not_autoplace no)
+			(effects
+				(font
+					(size 1.27 1.27)
+				)
+			)
+		)
+		(property "Description" "Solder Jumper, 2-pole, closed/bridged"
+			(at 137.16 78.74 0)
+			(hide yes)
+			(show_name no)
+			(do_not_autoplace no)
+			(effects
+				(font
+					(size 1.27 1.27)
+				)
+			)
+		)
+		(property "Mfr. No." ""
+			(at 137.16 73.66 0)
+			(hide yes)
+			(show_name no)
+			(do_not_autoplace no)
+			(effects
+				(font
+					(size 1.27 1.27)
+				)
+			)
+		)
+		(pin "2"
+		)
+		(pin "1"
+		)
+		(instances
+			(project "esp_home_sensor"
+				(path "/1b1bee14-8d82-405b-b99d-415549a137e6/74ba5f49-7b36-4eb7-9148-c1caa100b65a"
+					(reference "JP8")
+					(unit 1)
+				)
+			)
+		)
+	)
+	(symbol
 		(lib_id "power:GND")
 		(at 59.69 90.17 0)
@@
 			)
 		)
-		(property "Footprint" ""
+		(property "Footprint" "Jumper:SolderJumper-2_P1.3mm_Bridged2Bar_Pad1.0x1.5mm"
 			(at 78.74 140.97 0)
 			(hide yes)

Commit message: initial layout, power routing
Connections:
- net VOUT: no longer C2.1
- net ISET: now reaches R1.1, U1.2 (ISET)
- net VSET: now reaches R2.1, U1.7 (VSET)
- net OUT: now reaches JP8.1 (A), R3.2, R4.2, U1.8 (OUT)
- net OUT: now also C2.1
Changed lines of the file:
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@@
 	)
 	(junction
-		(at 147.32 73.66)
-		(diameter 0)
-		(color 0 0 0 0)
-	)
-	(junction
 		(at 125.73 92.71)
 		(diameter 0)
@@
 		(color 0 0 0 0)
 	)
+	(junction
+		(at 147.32 73.66)
+		(diameter 0)
+		(color 0 0 0 0)
+	)
 	(wire
 		(pts
@@
 	(wire
 		(pts
-			(xy 125.73 73.66) (xy 132.08 73.66)
+			(xy 125.73 73.66) (xy 147.32 73.66)
 		)
 		(stroke
@@
 	(wire
 		(pts
-			(xy 142.24 73.66) (xy 147.32 73.66)
+			(xy 68.58 80.01) (xy 68.58 76.2)
 		)
 		(stroke
@@
 	(wire
 		(pts
-			(xy 68.58 80.01) (xy 68.58 76.2)
+			(xy 152.4 73.66) (xy 147.32 73.66)
 		)
 		(stroke
@@
 	(wire
 		(pts
+			(xy 147.32 73.66) (xy 147.32 80.01)
+		)
+		(stroke
+			(width 0)
+			(type default)
+		)
+	)
+	(wire
+		(pts
 			(xy 82.55 151.13) (xy 85.09 151.13)
 		)
@@
 	(wire
 		(pts
-			(xy 152.4 73.66) (xy 147.32 73.66)
+			(xy 167.64 73.66) (xy 162.56 73.66)
 		)
 		(stroke
@@
 	(wire
 		(pts
-			(xy 147.32 73.66) (xy 147.32 80.01)
-		)
-		(stroke
-			(width 0)
-			(type default)
-		)
-	)
-	(wire
-		(pts
 			(xy 73.66 78.74) (xy 80.01 78.74)
 		)
@@
 		)
 	)
+	(label "VSET"
+		(at 107.95 76.2 180)
+		(effects
+			(font
+				(size 1.27 1.27)
+			)
+			(justify right bottom)
+		)
+	)
 	(label "STAT"
 		(at 107.95 81.28 180)
@@
 		)
 	)
+	(label "OUT"
+		(at 107.95 73.66 180)
+		(effects
+			(font
+				(size 1.27 1.27)
+			)
+			(justify right bottom)
+		)
+	)
+	(label "ISET"
+		(at 73.66 76.2 0)
+		(effects
+			(font
+				(size 1.27 1.27)
+			)
+			(justify left bottom)
+		)
+	)
 	(label "TS"
 		(at 73.66 78.74 0)
@@
 	(hierarchical_label "VOUT"
 		(shape output)
-		(at 152.4 73.66 0)
+		(at 167.64 73.66 0)
 		(effects
 			(font
@@
 		)
 	)
+	(netclass_flag ""
+		(length 2.54)
+		(shape round)
+		(at 125.73 73.66 0)
+		(fields_autoplaced yes)
+		(effects
+			(font
+				(size 1.27 1.27)
+			)
+			(justify left bottom)
+		)
+		(property "Klasy sieci" "Power"
+			(at 126.4285 71.12 0)
+			(show_name no)
+			(do_not_autoplace no)
+			(effects
+				(font
+					(size 1.27 1.27)
+				)
+				(justify left)
+			)
+		)
+		(property "Component Class" ""
+			(at 26.67 5.08 0)
+			(show_name no)
+			(do_not_autoplace no)
+			(effects
+				(font
+					(size 1.27 1.27)
+					(italic yes)
+				)
+			)
+		)
+	)
 	(symbol
 		(lib_id "Device:R")
@@
 	)
 	(symbol
-		(lib_id "Jumper:SolderJumper_2_Bridged")
-		(at 137.16 73.66 0)
-		(unit 1)
-		(body_style 1)
-		(exclude_from_sim no)
-		(in_bom no)
-		(on_board yes)
-		(in_pos_files yes)
-		(dnp no)
-		(fields_autoplaced yes)
-		(property "Reference" "JP8"
-			(at 137.16 67.31 0)
-			(show_name no)
-			(do_not_autoplace no)
-			(effects
-				(font
-					(size 1.27 1.27)
-				)
-			)
-		)
-		(property "Value" "SolderJumper_2_Bridged"
-			(at 137.16 69.85 0)
-			(show_name no)
-			(do_not_autoplace no)
-			(effects
-				(font
-					(size 1.27 1.27)
-				)
-			)
-		)
-		(property "Footprint" "Jumper:SolderJumper-2_P1.3mm_Bridged2Bar_Pad1.0x1.5mm"
-			(at 137.16 73.66 0)
-			(hide yes)
-			(show_name no)
-			(do_not_autoplace no)
-			(effects
-				(font
-					(size 1.27 1.27)
-				)
-			)
-		)
-		(property "Datasheet" ""
-			(at 137.16 80.01 0)
-			(hide yes)
-			(show_name no)
-			(do_not_autoplace no)
-			(effects
-				(font
-					(size 1.27 1.27)
-				)
-			)
-		)
-		(property "Description" "Solder Jumper, 2-pole, closed/bridged"
-			(at 137.16 78.74 0)
-			(hide yes)
-			(show_name no)
-			(do_not_autoplace no)
-			(effects
-				(font
-					(size 1.27 1.27)
-				)
-			)
-		)
-		(property "Mfr. No." ""
-			(at 137.16 73.66 0)
-			(hide yes)
-			(show_name no)
-			(do_not_autoplace no)
-			(effects
-				(font
-					(size 1.27 1.27)
-				)
-			)
-		)
-		(pin "2"
-		)
-		(pin "1"
-		)
-		(instances
-			(project "esp_home_sensor"
-				(path "/1b1bee14-8d82-405b-b99d-415549a137e6/74ba5f49-7b36-4eb7-9148-c1caa100b65a"
-					(reference "JP8")
-					(unit 1)
-				)
-			)
-		)
-	)
-	(symbol
 		(lib_id "power:GND")
 		(at 59.69 90.17 0)
@@
 					(unit 1)
 				)
+			)
+		)
+	)
+	(symbol
+		(lib_id "Jumper:SolderJumper_2_Bridged")
+		(at 157.48 73.66 0)
+		(unit 1)
+		(body_style 1)
+		(exclude_from_sim no)
+		(in_bom no)
+		(on_board yes)
+		(in_pos_files yes)
+		(dnp no)
+		(fields_autoplaced yes)
+		(property "Reference" "JP8"
+			(at 157.48 67.31 0)
+			(show_name no)
+			(do_not_autoplace no)
+			(effects
+				(font
+					(size 1.27 1.27)
+				)
+			)
+		)
+		(property "Value" "SolderJumper_2_Bridged"
+			(at 157.48 69.85 0)
+			(show_name no)
+			(do_not_autoplace no)
+			(effects
+				(font
+					(size 1.27 1.27)
+				)
+			)
+		)
+		(property "Footprint" "Jumper:SolderJumper-2_P1.3mm_Bridged2Bar_Pad1.0x1.5mm"
+			(at 157.48 73.66 0)
+			(hide yes)
+			(show_name no)
+			(do_not_autoplace no)
+			(effects
+				(font
+					(size 1.27 1.27)
+				)
+			)
+		)
+		(property "Datasheet" ""
+			(at 157.48 80.01 0)
+			(hide yes)
+			(show_name no)
+			(do_not_autoplace no)
+			(effects
+				(font
+					(size 1.27 1.27)
+				)
+			)
+		)
+		(property "Description" "Solder Jumper, 2-pole, closed/bridged"
+			(at 157.48 78.74 0)
+			(hide yes)
+			(show_name no)
+			(do_not_autoplace no)
+			(effects
+				(font
+					(size 1.27 1.27)
+				)
+			)
+		)
+		(property "Mfr. No." ""
+			(at 157.48 73.66 0)
+			(hide yes)
+			(show_name no)
+			(do_not_autoplace no)
+			(effects
+				(font
+					(size 1.27 1.27)
+				)
+			)
+		)
+		(pin "2"
+		)
+		(pin "1"
+		)
+		(instances
+			(project "esp_home_sensor"
+				(path "/1b1bee14-8d82-405b-b99d-415549a137e6/74ba5f49-7b36-4eb7-9148-c1caa100b65a"
+					(reference "JP8")
+					(unit 1)
+				)

Commit message: layout
Parts:
- renumbered JP6 to JP1, JP8 to JP2, R1 to R2, R6 to R3, R5 to R4, R3 to R5, R4 to R6, R2 to R7
Changed lines of the file:
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@@
 		(dnp no)
 		(fields_autoplaced yes)
-		(property "Reference" "R1"
+		(property "Reference" "R2"
 			(at 71.12 82.5499 0)
 			(show_name no)
@@
 			(project "esp_home_sensor"
 				(path "/1b1bee14-8d82-405b-b99d-415549a137e6/74ba5f49-7b36-4eb7-9148-c1caa100b65a"
-					(reference "R1")
+					(reference "R2")
 					(unit 1)
 				)
@@
 		(dnp no)
 		(fields_autoplaced yes)
-		(property "Reference" "R6"
+		(property "Reference" "R3"
 			(at 69.85 156.2099 0)
 			(show_name no)
@@
 			(project "esp_home_sensor"
 				(path "/1b1bee14-8d82-405b-b99d-415549a137e6/74ba5f49-7b36-4eb7-9148-c1caa100b65a"
-					(reference "R6")
+					(reference "R3")
 					(unit 1)
 				)
@@
 		(in_pos_files yes)
 		(dnp no)
-		(property "Reference" "#PWR06"
+		(property "Reference" "#PWR019"
 			(at 72.39 168.91 0)
 			(hide yes)
@@
 			(project "esp_home_sensor"
 				(path "/1b1bee14-8d82-405b-b99d-415549a137e6/74ba5f49-7b36-4eb7-9148-c1caa100b65a"
-					(reference "#PWR06")
+					(reference "#PWR019")
 					(unit 1)
 				)
@@
 		(dnp no)
 		(fields_autoplaced yes)
-		(property "Reference" "R4"
+		(property "Reference" "R6"
 			(at 116.84 96.52 90)
 			(show_name no)
@@
 			(project "esp_home_sensor"
 				(path "/1b1bee14-8d82-405b-b99d-415549a137e6/74ba5f49-7b36-4eb7-9148-c1caa100b65a"
-					(reference "R4")
+					(reference "R6")
 					(unit 1)
 				)
@@
 		(dnp no)
 		(fields_autoplaced yes)
-		(property "Reference" "R2"
+		(property "Reference" "R7"
 			(at 138.43 82.5499 0)
 			(show_name no)
@@
 			(project "esp_home_sensor"
 				(path "/1b1bee14-8d82-405b-b99d-415549a137e6/74ba5f49-7b36-4eb7-9148-c1caa100b65a"
-					(reference "R2")
+					(reference "R7")
 					(unit 1)
 				)
@@
 		(in_pos_files yes)
 		(dnp no)
-		(property "Reference" "#PWR02"
+		(property "Reference" "#PWR018"
 			(at 68.58 96.52 0)
 			(hide yes)
@@
 			(project "esp_home_sensor"
 				(path "/1b1bee14-8d82-405b-b99d-415549a137e6/74ba5f49-7b36-4eb7-9148-c1caa100b65a"
-					(reference "#PWR02")
+					(reference "#PWR018")
 					(unit 1)
 				)
@@
 		(in_pos_files yes)
 		(dnp no)
-		(property "Reference" "#PWR03"
+		(property "Reference" "#PWR017"
 			(at 59.69 96.52 0)
 			(hide yes)
@@
 			(project "esp_home_sensor"
 				(path "/1b1bee14-8d82-405b-b99d-415549a137e6/74ba5f49-7b36-4eb7-9148-c1caa100b65a"
-					(reference "#PWR03")
+					(reference "#PWR017")
 					(unit 1)
 				)
@@
 		(in_pos_files yes)
 		(dnp no)
-		(property "Reference" "#PWR01"
+		(property "Reference" "#PWR020"
 			(at 77.47 96.52 0)
 			(hide yes)
@@
 			(project "esp_home_sensor"
 				(path "/1b1bee14-8d82-405b-b99d-415549a137e6/74ba5f49-7b36-4eb7-9148-c1caa100b65a"
-					(reference "#PWR01")
+					(reference "#PWR020")
 					(unit 1)
 				)
@@
 		(dnp no)
 		(fields_autoplaced yes)
-		(property "Reference" "JP6"
+		(property "Reference" "JP1"
 			(at 78.74 134.62 0)
 			(show_name no)
@@
 			(project "esp_home_sensor"
 				(path "/1b1bee14-8d82-405b-b99d-415549a137e6/74ba5f49-7b36-4eb7-9148-c1caa100b65a"
-					(reference "JP6")
+					(reference "JP1")
 					(unit 1)
 				)
@@
 		(in_pos_files yes)
 		(dnp no)
-		(property "Reference" "#PWR07"
+		(property "Reference" "#PWR021"
 			(at 85.09 168.91 0)
 			(hide yes)
@@
 			(project "esp_home_sensor"
 				(path "/1b1bee14-8d82-405b-b99d-415549a137e6/74ba5f49-7b36-4eb7-9148-c1caa100b65a"
-					(reference "#PWR07")
+					(reference "#PWR021")
 					(unit 1)
 				)
@@
 		(in_pos_files yes)
 		(dnp no)
-		(property "Reference" "#PWR05"
+		(property "Reference" "#PWR023"
 			(at 147.32 96.52 0)
 			(hide yes)
@@
 			(project "esp_home_sensor"
 				(path "/1b1bee14-8d82-405b-b99d-415549a137e6/74ba5f49-7b36-4eb7-9148-c1caa100b65a"
-					(reference "#PWR05")
+					(reference "#PWR023")
 					(unit 1)
 				)
@@
 		(in_pos_files yes)
 		(dnp no)
-		(property "Reference" "#PWR04"
+		(property "Reference" "#PWR022"
 			(at 135.89 96.52 0)
 			(hide yes)
@@
 			(project "esp_home_sensor"
 				(path "/1b1bee14-8d82-405b-b99d-415549a137e6/74ba5f49-7b36-4eb7-9148-c1caa100b65a"
-					(reference "#PWR04")
+					(reference "#PWR022")
 					(unit 1)
 				)
@@
 		(dnp no)
 		(fields_autoplaced yes)
-		(property "Reference" "R5"
+		(property "Reference" "R4"
 			(at 78.74 144.78 90)
 			(show_name no)
@@
 			(project "esp_home_sensor"
 				(path "/1b1bee14-8d82-405b-b99d-415549a137e6/74ba5f49-7b36-4eb7-9148-c1caa100b65a"
-					(reference "R5")
+					(reference "R4")
 					(unit 1)
 				)
@@
 		(dnp no)
 		(fields_autoplaced yes)
-		(property "Reference" "JP8"
+		(property "Reference" "JP2"
 			(at 157.48 67.31 0)
 			(show_name no)
@@
 			(project "esp_home_sensor"
 				(path "/1b1bee14-8d82-405b-b99d-415549a137e6/74ba5f49-7b36-4eb7-9148-c1caa100b65a"
-					(reference "JP8")
+					(reference "JP2")
 					(unit 1)
 				)
@@
 		(dnp no)
 		(fields_autoplaced yes)
-		(property "Reference" "R3"
+		(property "Reference" "R5"
 			(at 116.84 86.36 90)
 			(show_name no)
@@
 			(project "esp_home_sensor"
 				(path "/1b1bee14-8d82-405b-b99d-415549a137e6/74ba5f49-7b36-4eb7-9148-c1caa100b65a"
-					(reference "R3")
-					(unit 1)
-				)
+					(reference "R5")
+					(unit 1)
+				)

Commit message: in production
Parts:
- C1, C2: Mfr. No. (none) -> GRM155R61E105MA12D
- D1, D2: Mfr. No. (none) -> LTST-C281KRKT
- R2: Mfr. No. (none) -> RC0402FR-07680RL
- R5, R6: Mfr. No. (none) -> RC0402FR-0710KL
- R7: Mfr. No. (none) -> RC0402FR-0727KL
- TH1: value NTCSP163JF103FT1H -> NTCG103JF103FT1; Mfr. No. NTCSP163JF103FT1H -> NTCG103JF103FT1
- U1: Mfr. No. BQ25170JDSGR -> BQ25170JDSGR
Changed lines of the file:
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@@
 			)
 		)
-		(property "Mfr. No." ""
+		(property "Mfr. No." "RC0402FR-07680RL"
 			(at 68.58 83.82 0)
 			(hide yes)
@@
 			)
 		)
-		(property "Mfr. No." ""
+		(property "Mfr. No." "GRM155R61E105MA12D"
 			(at 59.69 83.82 0)
 			(hide yes)
@@
 			)
 		)
-		(property "Mfr. No." ""
+		(property "Mfr. No." "LTST-C281KRKT"
 			(at 107.95 92.71 0)
 			(hide yes)
@@
 			)
 		)
-		(property "Mfr. No." "BQ25170JDSGR "
+		(property "Mfr. No." "BQ25170JDSGR"
 			(at 90.17 76.2 0)
 			(hide yes)
@@
 			)
 		)
-		(property "Mfr. No." ""
+		(property "Mfr. No." "RC0402FR-0710KL"
 			(at 116.84 102.87 90)
 			(hide yes)
@@
 			)
 		)
-		(property "Mfr. No." ""
+		(property "Mfr. No." "RC0402FR-0727KL"
 			(at 135.89 83.82 0)
 			(hide yes)
@@
 			)
 		)
-		(property "Mfr. No." ""
+		(property "Mfr. No." "LTST-C281KRKT"
 			(at 107.95 102.87 0)
 			(hide yes)
@@
 			)
 		)
-		(property "Mfr. No." ""
+		(property "Mfr. No." "GRM155R61E105MA12D"
 			(at 147.32 83.82 0)
 			(hide yes)
@@
 			)
 		)
-		(property "Value" "NTCSP163JF103FT1H"
+		(property "Value" "NTCG103JF103FT1"
 			(at 87.63 159.0674 0)
 			(show_name no)
@@
 			)
 		)
-		(property "Mfr. No." "NTCSP163JF103FT1H"
+		(property "Mfr. No." "NTCG103JF103FT1"
 			(at 85.09 157.48 0)
 			(hide yes)
@@
 			)
 		)
-		(property "Mfr. No." ""
+		(property "Mfr. No." "RC0402FR-0710KL"
 			(at 116.84 92.71 90)
 			(hide yes)

Commit message: az
Parts:
- U1: Down_current (none) -> 350n; Supply_current (none) -> N/A
